Commit message: Add files via upload

File: ras_robot_simulation/urdf/roda.xacro (robot description, xacro)
@@ -28,4 +28,5 @@
             <axis xyz="0 1 0"/>
             <limit effort="100" velocity="100"/>
+            <dynamics damping="2.0" friction="0.1"/>
         </joint>
         <gazebo reference="${prefix}_roda_link">

File: ras_robot_simulation/urdf/roda_boba.xacro (robot description, xacro)
@@ -49,6 +49,6 @@
         <gazebo reference="${prefix}_roda_boba_link">
             <material>Gazebo/DarkGrey</material>
-            <mu1>0.0</mu1>
-            <mu2>0.0</mu2>
+            <mu1>0.1</mu1>
+            <mu2>0.1</mu2>
             <kp>1000000.0</kp>
             <kd>10.0</kd>
